File: choc/horizon-choc.kicad_pcb (KiCad board)
At the start: 2 copper layers, 252 x 68 mm, 63 parts, among them SW1 SW_Push, SW10 SW_Push, SW11 SW_Push, SW12 SW_Push, SW13 SW_Push, SW14 SW_Push, SW15 SW_Push, SW16 SW_Push, SW17 SW_Push, SW18 SW_Push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

Commit message: updated pcb
Parts:
- added REF**: STAB_choc_2u, marbastlib-choc-untested:STAB_choc_2u, F.Cu at (112.0, 130.4)
- added REF**: STAB_choc_2u, marbastlib-choc-untested:STAB_choc_2u, F.Cu at (112.0, 131.9)
- added REF**: SW_choc_1u, marbastlib-choc:SW_choc_1u, F.Cu at (112.0, 130.5)
