File: pcb/RP2040_tmp.kicad_pcb (KiCad board)
At the start: 2 copper layers, 34 parts, among them J0 USB_C_Receptacle_USB2.0, J1 BREAKOUT, J2 Conn_01x03_Male, J4 Conn_01x01_Male, SW0 RESET, SW2 RESET, U1 NCP1117-3.3_SOT223, U2 W25Q128JVS, U3 RP2040, U44 SRV05-4, Y0 12MHZ Crystal

Commit message: updated pcb
Parts:
- added D1: BAV70, Package_TO_SOT_SMD:SOT-23, F.Cu at (99.0, 44.1)
- added D10: BAV70, Package_TO_SOT_SMD:SOT-23, F.Cu at (108.0, 53.2)
- added D11: BAV70, Package_TO_SOT_SMD:SOT-23, F.Cu at (121.3, 39.5)
- added D12: BAV70, Package_TO_SOT_SMD:SOT-23, F.Cu at (130.2, 39.5)
- added D13: BAV70, Package_TO_SOT_SMD:SOT-23, F.Cu at (116.8, 44.1)
- added D14: BAV70, Package_TO_SOT_SMD:SOT-23, F.Cu at (112.4, 53.2)
- added D15: BAV70, Package_TO_SOT_SMD:SOT-23, F.Cu at (99.0, 53.2)
- added D16: BAV70, Package_TO_SOT_SMD:SOT-23, F.Cu at (116.8, 53.2)
- added D17: BAV70, Package_TO_SOT_SMD:SOT-23, F.Cu at (103.5, 39.5)
- added D18: BAV70, Package_TO_SOT_SMD:SOT-23, F.Cu at (103.5, 48.6)
- added D19: BAV70, Package_TO_SOT_SMD:SOT-23, F.Cu at (112.4, 44.1)
- added D2: BAV70, Package_TO_SOT_SMD:SOT-23, F.Cu at (116.8, 48.6)
- added D20: BAV70, Package_TO_SOT_SMD:SOT-23, F.Cu at (103.5, 53.2)
- added D21: BAV70, Package_TO_SOT_SMD:SOT-23, F.Cu at (103.5, 44.1)
- added D22: BAV70, Package_TO_SOT_SMD:SOT-23, F.Cu at (125.8, 39.5)
- added D23: BAV70, Package_TO_SOT_SMD:SOT-23, F.Cu at (112.4, 39.5)
- added D24: BAV70, Package_TO_SOT_SMD:SOT-23, F.Cu at (99.0, 39.5)
- added D25: BAV70, Package_TO_SOT_SMD:SOT-23, F.Cu at (108.0, 48.6)
- added D26: BAV70, Package_TO_SOT_SMD:SOT-23, F.Cu at (112.4, 48.6)
- added D27: BAV70, Package_TO_SOT_SMD:SOT-23, F.Cu at (130.2, 44.1)
- added D3: BAV70, Package_TO_SOT_SMD:SOT-23, F.Cu at (116.8, 39.5)
- added D4: BAV70, Package_TO_SOT_SMD:SOT-23, F.Cu at (108.0, 44.1)
- added D5: BAV70, Package_TO_SOT_SMD:SOT-23, F.Cu at (99.0, 48.6)
- added D6: BAV70, Package_TO_SOT_SMD:SOT-23, F.Cu at (121.3, 44.1)
- added D7: BAV70, Package_TO_SOT_SMD:SOT-23, F.Cu at (125.8, 44.1)
- added D8: BAV70, Package_TO_SOT_SMD:SOT-23, F.Cu at (121.3, 48.6)
- added D9: BAV70, Package_TO_SOT_SMD:SOT-23, F.Cu at (108.0, 39.5)
- added H1: Hole_Pad, horizon-footprints:Mount_M2, F.Cu at (40.0, 88.0)
- added H2: Hole_Pad, horizon-footprints:Mount_M2, F.Cu at (256.0, 88.0)
- added H3: Hole_Pad, horizon-footprints:Mount_M2, F.Cu at (40.0, 122.0)
- added H4: Hole_Pad, horizon-footprints:Mount_M2, F.Cu at (256.0, 122.0)
- added H5: Hole_Pad, horizon-footprints:Mount_M2, F.Cu at (134.5, 75.5)
- added H6: Hole_Pad, horizon-footprints:Mount_M2, F.Cu at (161.5, 75.5)
- added H7: Hole_Pad, horizon-footprints:Mount_M2, F.Cu at (134.5, 100.5)
- added H8: Hole_Pad, horizon-footprints:Mount_M2, F.Cu at (161.5, 100.5)
- added K1: KEYSW, keyswitches:Kailh_socket_PG1350_optional, F.Cu at (31.0, 79.5)
- added K10: KEYSW, keyswitches:Kailh_socket_PG1350_optional, F.Cu at (67.0, 96.5)
- added K11: KEYSW, keyswitches:Kailh_socket_PG1350_optional, F.Cu at (67.0, 113.5)
- added K12: KEYSW, keyswitches:Kailh_socket_PG1350_optional, F.Cu at (67.0, 130.5)
- added K13: KEYSW, keyswitches:Kailh_socket_PG1350_optional, F.Cu at (85.0, 79.5)
- added K14: KEYSW, keyswitches:Kailh_socket_PG1350_optional, F.Cu at (85.0, 96.5)
- added K15: KEYSW, keyswitches:Kailh_socket_PG1350_optional, F.Cu at (85.0, 113.5)
- added K16: KEYSW, keyswitches:Kailh_socket_PG1350_optional, F.Cu at (85.0, 130.5)
- added K17: KEYSW, keyswitches:Kailh_socket_PG1350_optional, F.Cu at (103.0, 79.5)
- added K18: KEYSW, keyswitches:Kailh_socket_PG1350_optional, F.Cu at (103.0, 96.5)
- added K19: KEYSW, keyswitches:Kailh_socket_PG1350_optional, F.Cu at (103.0, 113.5)
- added K2: KEYSW, keyswitches:Kailh_socket_PG1350_optional, F.Cu at (31.0, 96.5)
- added K20: KEYSW, keyswitches:Kailh_socket_PG1350_optional, F.Cu at (103.0, 130.5)
- added K21: KEYSW, keyswitches:Kailh_socket_PG1350_optional, F.Cu at (121.0, 79.5)
- added K22: KEYSW, keyswitches:Kailh_socket_PG1350_optional, F.Cu at (121.0, 96.5)
- added K23: KEYSW, keyswitches:Kailh_socket_PG1350_optional, F.Cu at (121.0, 113.5)
- added K24: KEYSW, keyswitches:Kailh_socket_PG1350_optional, F.Cu at (121.0, 130.5)
- added K25: KEYSW, keyswitches:Kailh_socket_PG1350_optional, F.Cu at (139.0, 113.5)
- added K26: KEYSW, keyswitches:Kailh_socket_PG1350_optional, F.Cu at (139.0, 130.5)
- added K27: KEYSW, keyswitches:Kailh_socket_PG1350_optional, F.Cu at (157.0, 113.5)
- added K28: KEYSW, keyswitches:Kailh_socket_PG1350_optional, F.Cu at (157.0, 130.5)
- added K29: KEYSW, keyswitches:Kailh_socket_PG1350_optional, F.Cu at (175.0, 79.5)
- added K3: KEYSW, keyswitches:Kailh_socket_PG1350_optional, F.Cu at (31.0, 113.5)
- added K30: KEYSW, keyswitches:Kailh_socket_PG1350_optional, F.Cu at (175.0, 96.5)
- added K31: KEYSW, keyswitches:Kailh_socket_PG1350_optional, F.Cu at (175.0, 113.5)
- added K32: KEYSW, keyswitches:Kailh_socket_PG1350_optional, F.Cu at (175.0, 130.5)
- added K33: KEYSW, keyswitches:Kailh_socket_PG1350_optional, F.Cu at (193.0, 79.5)
- added K34: KEYSW, keyswitches:Kailh_socket_PG1350_optional, F.Cu at (193.0, 96.5)
- added K35: KEYSW, keyswitches:Kailh_socket_PG1350_optional, F.Cu at (193.0, 113.5)
- added K36: KEYSW, keyswitches:Kailh_socket_PG1350_optional, F.Cu at (193.0, 130.5)
- added K37: KEYSW, keyswitches:Kailh_socket_PG1350_optional, F.Cu at (211.0, 79.5)
- added K38: KEYSW, keyswitches:Kailh_socket_PG1350_optional, F.Cu at (211.0, 96.5)
- added K39: KEYSW, keyswitches:Kailh_socket_PG1350_optional, F.Cu at (211.0, 113.5)
- added K4: KEYSW, keyswitches:Kailh_socket_PG1350_optional, F.Cu at (31.0, 130.5)
- added K40: KEYSW, keyswitches:Kailh_socket_PG1350_optional, F.Cu at (211.0, 130.5)
- added K41: KEYSW, keyswitches:Kailh_socket_PG1350_optional, F.Cu at (229.0, 79.5)
- added K42: KEYSW, keyswitches:Kailh_socket_PG1350_optional, F.Cu at (229.0, 96.5)
- added K43: KEYSW, keyswitches:Kailh_socket_PG1350_optional, F.Cu at (229.0, 113.5)
- added K44: KEYSW, keyswitches:Kailh_socket_PG1350_optional, F.Cu at (229.0, 130.5)
- added K45: KEYSW, keyswitches:Kailh_socket_PG1350_optional, F.Cu at (247.0, 79.5)
- added K46: KEYSW, keyswitches:Kailh_socket_PG1350_optional, F.Cu at (247.0, 96.5)
- added K47: KEYSW, keyswitches:Kailh_socket_PG1350_optional, F.Cu at (247.0, 113.5)
- added K48: KEYSW, keyswitches:Kailh_socket_PG1350_optional, F.Cu at (247.0, 130.5)
- added K49: KEYSW, keyswitches:Kailh_socket_PG1350_optional, F.Cu at (265.0, 79.5)
- added K5: KEYSW, keyswitches:Kailh_socket_PG1350_optional, F.Cu at (49.0, 79.5)
- added K50: KEYSW, keyswitches:Kailh_socket_PG1350_optional, F.Cu at (265.0, 96.5)
- added K51: KEYSW, keyswitches:Kailh_socket_PG1350_optional, F.Cu at (265.0, 113.5)
- added K52: KEYSW, keyswitches:Kailh_socket_PG1350_optional, F.Cu at (265.0, 130.5)
- added K6: KEYSW, keyswitches:Kailh_socket_PG1350_optional, F.Cu at (49.0, 96.5)
- added K7: KEYSW, keyswitches:Kailh_socket_PG1350_optional, F.Cu at (49.0, 113.5)
- added K8: KEYSW, keyswitches:Kailh_socket_PG1350_optional, F.Cu at (49.0, 130.5)
- added K9: KEYSW, keyswitches:Kailh_socket_PG1350_optional, F.Cu at (67.0, 79.5)
- added LED1: WS2812B, WS2812B:WS2812B, F.Cu at (185.7, 54.9)
- added LED2: WS2812B, WS2812B:WS2812B, F.Cu at (195.5, 46.6)
- added LED3: WS2812B, WS2812B:WS2812B, F.Cu at (191.8, 54.9)
- added LOGO1: Logo-Bottom, horizon-footprints:Logo_Horizon_Small, B.Cu at (148.0, 87.5)
- added LOGO2: Logo-Top, horizon-footprints:Logo_Horizon_H, F.Cu at (148.0, 88.0)
- added REF**: STAB_choc_2u, marbastlib-choc-untested:STAB_choc_2u, F.Cu at (112.0, 130.4)
- added REF**: STAB_choc_2u, marbastlib-choc-untested:STAB_choc_2u, F.Cu at (112.0, 131.9)
- added SW1: RotaryEncoder_Switch, Keebio-Parts:RotaryEncoder_Alps_EC11E-Switch_Vertical_H20mm, F.Cu at (223.7, 50.4)
- added SW3: RotaryEncoder_Switch, Keebio-Parts:RotaryEncoder_Alps_EC11E-Switch_Vertical_H20mm, F.Cu at (227.0, 27.1)
- added Ureserved1: larger footprint, more mA available, Package_TO_SOT_SMD:SOT-223-3_TabPin2, F.Cu at (177.5, 57.1)
- U1: value NCP1117-3.3_SOT223 -> XC6206 smaller footprint; footprint Package_TO_SOT_SMD:SOT-223-3_TabPin2 -> Package_TO_SOT_SMD:SOT-23
- moved SW0 136.3 mm to (151.9, 99.4)
- moved U1 133.2 mm to (157.7, 80.3), turned to -90 degrees
- moved J0 129.3 mm to (148.0, 73.2), turned to 180 degrees
- moved F0 128.9 mm to (154.6, 75.3), turned to -90 degrees
- moved C3 128.5 mm to (155.2, 90.7), turned to -45 degrees
- moved C2 127.2 mm to (150.8, 95.1), turned to 135 degrees
- moved C5 126.5 mm to (160.4, 96.2)
- moved U2 125.6 mm to (134.5, 88.0), turned to 90 degrees
- moved SW2 122.2 mm to (142.4, 99.2)
- moved C1 121.9 mm to (160.5, 80.3), turned to 90 degrees
- moved Y0 121.7 mm to (153.0, 92.9), turned to -135 degrees
- moved R1 119.6 mm to (156.7, 99.1)
- moved C4 119.3 mm to (152.8, 80.3), turned to 90 degrees
- moved R5 117.9 mm to (156.7, 89.2), turned to -45 degrees
- moved U3 116.1 mm to (148.0, 88.0), turned to 45 degrees
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Connections:
- U3 pad 2: rot_2_l -> unconnected-(U3-Pad2)
- U3 pad 3: rot_2_r -> unconnected-(U3-Pad3)
- U3 pad 4: rot_1_l -> unconnected-(U3-Pad4)
- U3 pad 5: rot_1_r -> unconnected-(U3-Pad5)
- U44 pad 3: /USB_D+ -> /USB_D-
- U44 pad 4: unconnected-(U44-Pad4) -> /USB_D+
- U44 pad 6: /USB_D- -> unconnected-(U44-Pad6)
Routing:
- net GND: track 0.00 -> 65.5 mm, vias 0 -> 2
- net +5V: track 0.00 -> 33.8 mm, vias 0 -> 4
- net +3V3: track 0.00 -> 21.0 mm
- net /USB_D+: track 0.00 -> 19.1 mm, vias 0 -> 1
- net VBUS: track 0.00 -> 15.5 mm
- net /USB_D-: track 0.00 -> 14.0 mm
- net Net-(J0-PadA5): track 0.00 -> 10.8 mm
- net /SWD: track 0.00 -> 8.17 mm, vias 0 -> 1
- net /XIN: track 0.00 -> 7.61 mm
- net /XOUT: track 0.00 -> 7.15 mm
- net Net-(J0-PadB5): track 0.00 -> 6.04 mm
- net /SWCLK: track 0.00 -> 5.37 mm, vias 0 -> 1
- net Net-(C3-Pad1): track 0.00 -> 4.88 mm
- net /RUN: track 0.00 -> 0.81 mm
- added copper zone on F.Cu, net GND
Other:
- board outline added: 252 x 68 mm
- rule pad_to_mask_clearance: 0 -> 0.051
- board text added: "JLCJLCJLCJLC"
- board text added: "github.com/skarrmann/horizon"
- board text added: "rev2.3 | Choc"
