File: pcb/RP2040_tmp.kicad_sch (KiCad schematic)
At the start: 35 parts, among them J0 USB_C_Receptacle_USB2.0, J1 BREAKOUT, J2 Conn_01x03_Male, J4 Conn_01x01_Male, SW0 RESET, SW2 RESET, U1 XC6206 smaller footprint, U1 larger footprint, more mA ava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, U2 W25Q128JVS, U3 RP2040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

Commit message: updated pcb
Parts:
- added LED1, LED2, LED3: WS2812B, WS2812B:WS2812B, symbol cipulot_parts:WS2812B
- renumbered U1 to Ureserved1
Connections:
- net +5V: now also LED1.1 (VCC), LED2.1 (VCC), LED3.1 (VCC)
- net GND: now also LED1.3 (GND), LED2.3 (GND), LED3.3 (GND)
- net LED_GLOW: now also LED1.4 (DIN)
- net USB_D+: now also U44.4 (IO3); no longer U44.3 (IO2)
- net USB_D-: now also U44.3 (IO2); no longer U44.6 (IO4)
- net rot_1_l: no longer names the net of U3.4 (GPIO2)
- net rot_1_r: no longer names the net of U3.5 (GPIO3)
- net rot_2_l: no longer names the net of U3.2 (GPIO0)
- net rot_2_r: no longer names the net of U3.3 (GPIO1)
- new net: LED1.2 (DOUT), LED2.4 (DIN)
- new net: LED2.2 (DOUT), LED3.4 (DIN)

Commit message: updated pcb
added onboard mcu
included silkscreen resembling sun and SOHO
added files for assembly with jlcpcb
Parts:
- removed C14, C7: 100n, Capacitor_SMD:C_0805_2012Metric, symbol Device:C
- removed Ureserved1: larger footprint, more mA available, Package_TO_SOT_SMD:SOT-223-3_TabPin2, symbol Regulator_Linear:NCP1117-3.3_SOT223
- J2: footprint Connector_PinSocket_1.27mm:PinSocket_1x03_P1.27mm_Vertical -> Connector_PinSocket_2.54mm:PinSocket_1x03_P2.54mm_Vertical
- LED1, LED2, LED3: footprint WS2812B:WS2812B -> weteor_library:SK6812_4020
- SW0, SW2: footprint Keebio-Parts:SW_SPST_TL3342 -> weteor_library:SMD_GT-H0065-L1; LCSC C2886894 -> C778132
Connections:
- net ROW4 is gone; now on net COL7: U3.16 (GPIO13)
- net COL0: now also U3.36 (GPIO24); no longer U3.37 (GPIO25)
- net COL1: now also U3.37 (GPIO25); no longer U3.36 (GPIO24)
- net COL10: now also U3.29 (GPIO18); no longer U3.18 (GPIO15)
- net COL11: now also U3.30 (GPIO19); no longer U3.17 (GPIO14)
- net COL12: now also U3.31 (GPIO20); no longer U3.15 (GPIO12)
- net COL13: now also U3.32 (GPIO21); no longer U3.14 (GPIO11)
- net COL2: now also U3.4 (GPIO2); no longer U3.35 (GPIO23)
- net COL3: now also U3.5 (GPIO3); no longer U3.34 (GPIO22)
- net COL4: now also U3.6 (GPIO4); no longer U3.32 (GPIO21)
- net COL5: now also U3.9 (GPIO7); no longer U3.31 (GPIO20)
- net COL6: now also U3.35 (GPIO23); no longer U3.30 (GPIO19)
- net COL7: no longer U3.29 (GPIO18)
- net ENC_2_LFT: now also U3.18 (GPIO15)
- net ENC_2_RGT: now also U3.17 (GPIO14)
- net LED_GLOW: no longer J2.3 (Pin_3)
- net ROW0: now also U3.34 (GPIO22); no longer U3.7 (GPIO5)
- net ROW1: now also U3.2 (GPIO0); no longer U3.6 (GPIO4)
- net ROW2: now also U3.3 (GPIO1); no longer U3.9 (GPIO7)
- net ROW3: now also U3.7 (GPIO5); no longer U3.12 (GPIO9)
- net LED_BREAKOUT: now reaches LED3.2 (DOUT)
- net LED_BREAKOUT: now also J2.3 (Pin_3)
- net COL14: no longer names the net of U3.13 (GPIO10)

Commit message: fixed issue of pcb, added assembly files for jlc
Parts:
- U1: LCSC C3015484 -> C347376
Changed lines of the file:
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@@
       (effects (font (size 1.27 1.27)) hide)
     )
-    (property "LCSC" "C3015484" (id 4) (at 74.93 176.53 0)
+    (property "LCSC" "C347376" (id 4) (at 74.93 176.53 0)
       (effects (font (size 1.27 1.27)) hide)
     )
